File: Kicad_bin/DTI_Cube_Proto.kicad_sch (KiCad schematic)
At the start: 23 parts

Commit message: Schemy boi
Parts:
- added R1, R2: 10k, symbol Device:R
- A1: renamed from A?; value (none) -> SD_Card_Module; footprint (none) -> Charleslabs_Parts:SD_Card_Module
- C1: renamed from C?; value (none) -> 0.1uF
- C3: renamed from C?; value (none) -> 10uF
- C5: renamed from C?; value (none) -> 220uF
- D1: renamed from D?; value (none) -> WS2812B; footprint (none) -> LED_SMD:LED_WS2812B_PLCC4_5.0x5.0mm_P3.2mm
- IC1: renamed from U?; value (none) -> DOIT-ESP32-DEVKIT-V1 (30 GPIO)
- LS1: renamed from LS?; value (none) -> 4R Speaker
- PS1: renamed from PS?; value (none) -> 12A LED PSU; footprint (none) -> Converter_ACDC:Converter_ACDC_MeanWell_IRM-60-xx_THT
- R3: renamed from R?; value (none) -> 1.2k
- R4: renamed from R?; value (none) -> 10R
- RV1: renamed from RV?; value (none) -> 10k
- SW1: renamed from SW?; value (none) -> SW_Push
- U1: renamed from U?; value (none) -> HC-SR04
- U3: renamed from U?; value (none) -> LM386
- gave numbers to parts that had none: 9
Connections:
- net GND: now also R1.2, R2.2
- net GPIO 27: now reaches D1.4 (DIN)
- net GPIO 27: now also IC1.10 (GPIO27)
- net at IC1.24 (GPIO15), SW1.1, SW2.1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: now also R2.1
- net at IC1.11 (GPIO14), U1.3 (ECHO): now also R1.1
- net GPIO 21: now reaches IC1.32 (GPIO21)
- net GPIO 21: now also RV1.1
Other:
- company: (none) -> JVWCSY ☆
- title: (none) -> DTI Staircase Cube
- moved on the sheet: A1, C1, C2, C3, C4, C5, D1, D2, D3, D4, D5, D6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

Commit message: A lot of changes, from a modded DAC_Audio library, to the test file for it, to the proto_3 changes
Parts:
- added D? (x6): WS2812B, LED_SMD:LED_WS2812B_PLCC4_5.0x5.0mm_P3.2mm, symbol LED:WS2812B
- added D? (x2): 1N4148, Diode_THT:D_DO-35_SOD27_P7.62mm_Horizontal, symbol Diode:1N4148
- PS1: value 12A LED PSU -> (none)
Connections:
- net +5V: now also D?.1 (VDD), D?.1 (VDD), D?.1 (VDD), D?.1 (VDD), D?.1 (VDD), D?.2 (A), D?.2 (A); no longer D1.1 (VDD)
- net GND: now also D?.3 (VSS), D?.3 (VSS), D?.3 (VSS), D?.3 (VSS), D?.3 (VSS), D?.3 (VSS)
- net GPIO 25: now reaches IC1.8 (GPIO25)
- net GPIO 25: now also RV1.1
- net GPIO 26: now reaches IC1.9 (GPIO26)
- net GPIO 26: now also D?.4 (DIN)
- net GPIO 21: no longer names the net of IC1.32 (GPIO21)
- net GPIO 21: no longer RV1.1
- new net: D?.1 (K), D?.1 (VDD)
- new net: D?.2 (DOUT), D?.4 (DIN) (x4)
- new net: D1.1 (VDD), D?.1 (K)
Other:
- note added: "Sacrifical Pixel"
- moved on the sheet: A1, C1, C2, C3, C4, C5, D1, D2, D3, D4, D5, D6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
